File: LCD-LiDAR-SD-Hat/Teensy-LCD-LiDAR-Hat.kicad_pcb (KiCad board)
At the start: 2 copper layers, 80 x 36.2 mm, 16 parts, among them J1 TEENSY3.2-72MHz, J2 LIDAR-LITE, J3 MICRO-SD

Commit message: Added board outline to assembly diagrams.
Other:
- board text added: "8/13/16"
- board text added: "LCD-LiDAR-SD Teensy Hat v1.0"
Changed lines of the file:
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@@
     (links 49)
     (no_connects 0)
-    (area 97.527699 97.028 178.077541 133.632621)
+    (area 97.527699 91.845 178.584285 137.725)
     (thickness 1.6)
-    (drawings 15)
+    (drawings 21)
     (tracks 140)
     (zones 0)
@@
   )
   (setup
-    (last_trace_width 0.3302)
+    (last_trace_width 0.25)
     (user_trace_width 0.1524)
     (user_trace_width 0.254)
@@
     (visible_elements FFFEDF7D)
     (pcbplotparams
-      (layerselection 0x3d0fc_80000001)
+      (layerselection 0x30000_00000000)
       (usegerberextensions true)
       (excludeedgelayer true)
@@
     (pad G4 smd rect (at 5.0514 3.95 270) (size 1 0.7) (layers F.Cu F.Paste F.Mask))
   )
+  (gr_text "8/13/16 " (at 172.72 136.525) (layer F.Fab)
+    (effects (font (size 1.5 1.5) (thickness 0.3)))
+  )
+  (gr_text "LCD-LiDAR-SD Teensy Hat v1.0" (at 158.75 93.345) (layer F.Fab)
+    (effects (font (size 1.5 1.5) (thickness 0.3)))
+  )
+  (gr_line (start 177.8 133.985) (end 177.8 97.155) (layer F.Fab) (width 0.2))
+  (gr_line (start 97.79 133.985) (end 177.8 133.985) (layer F.Fab) (width 0.2))
+  (gr_line (start 97.79 97.155) (end 97.79 133.985) (layer F.Fab) (width 0.2))
+  (gr_line (start 177.8 97.155) (end 97.79 97.155) (layer F.Fab) (width 0.2))
   (gr_text 16 (at 128.524 100.076) (layer F.SilkS)
     (effects (font (size 1.27 1.27) (thickness 0.254)))
   )
-  (gr_text 1 (at 172.212 99.822 360) (layer F.SilkS)
+  (gr_text 1 (at 172.212 99.822) (layer F.SilkS)
     (effects (font (size 1.27 1.27) (thickness 0.254)))
   )
