File: 7-Segment-Hat/hardware/Teensy-7-Segment-Hat.kicad_pcb (KiCad board)
At the start: 2 copper layers, 37.1 x 18 mm, 7 parts, among them J1 TEENSY3.2-72MHz-SIMPLE, J3 MICRO-SD

Commit message: Adjusted code location. Added photos.
Parts:
- moved LED1 2.54 mm to (137.0, 84.1)
- turned R2 to 0 degrees
- turned R3 to 0 degrees
- turned R4 to 0 degrees
Routing:
- net Net-(LED1-Pad8): track 3.06 -> 5.60 mm
- net Net-(LED1-Pad6): track 2.74 -> 3.55 mm
- net /DIGIT2: track 5.09 -> 5.76 mm
- net /DIGIT3: track 5.19 -> 5.82 mm
Other:
- board text added: "Quad 7-Segment Display Teensy Hat v1.1"
- board text removed: "Quad 7-Segment Display Teensy Hat v1.0"
